Commit message: update mesh path in urrf file

File: urdf/karl/karl.urdf (robot description, URDF)
Before this commit: robot karl, 27 links, 26 joints
Links:
- link base_link: geometry visual mesh filename=file:///mesh/karl/karl.obj
- link rack: geometry visual mesh filename=file:///mesh/karl/rack.obj

File: urdf/shuttle/shuttle.urdf (robot description, URDF)
Before this commit: robot shuttle, 5 links, 4 joints
Links:
- link base_link: geometry visual mesh filename=file:///mesh/shuttle/shuttle.obj
- link wheel_fl: geometry visual mesh filename=file:///mesh/shuttle/shuttle_wheel.obj
- link wheel_fr: geometry visual mesh filename=file:///mesh/shuttle/shuttle_wheel.obj
- link wheel_rl: geometry visual mesh filename=file:///mesh/shuttle/shuttle_wheel.obj
- link wheel_rr: geometry visual mesh filename=file:///mesh/shuttle/shuttle_wheel.obj
